Commit message: fix: correct wheel joint names for consistency in configuration

File: src/vesc_nexus/urdf/robot.urdf.xacro (robot description, xacro)
@@ -7,5 +7,5 @@
       <param name="wheel_radius">0.115</param>
     </hardware>
-    <joint name="front_left_wheel" type="continuous">
+    <joint name="left_front_wheel" type="continuous">
       <command_interface name="velocity"/>
       <state_interface name="velocity"/>
@@ -16,5 +16,5 @@
       <param name="wheel_radius">0.115</param>
     </joint>
-    <joint name="front_right_wheel" type="continuous">
+    <joint name="right_front_wheel" type="continuous">
       <command_interface name="velocity"/>
       <state_interface name="velocity"/>
@@ -25,5 +25,5 @@
       <param name="wheel_radius">0.115</param>
     </joint>
-    <joint name="rear_left_wheel" type="continuous">
+    <joint name="left_rear_wheel" type="continuous">
       <command_interface name="velocity"/>
       <state_interface name="velocity"/>
@@ -34,5 +34,5 @@
       <param name="wheel_radius">0.115</param>
     </joint>
-    <joint name="rear_right_wheel" type="continuous">
+    <joint name="right_rear_wheel" type="continuous">
       <command_interface name="velocity"/>
       <state_interface name="velocity"/>
